File: RaSK_Generic-Rocket-Logger.sch (KiCad schematic (older format))
At the start: 51 parts, among them J1 SD_Card, J2 TWE_Writer, J3 GS2, J4 Mount, J5 Mount, J6 Mount, J7 Mount, P1 STLINK_SWD, P2 KRC_PSoCWriter, P3 TRIGOUT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

Commit message: add buzzer out and trigger pin to port
Parts:
- removed P3: TRIGOUT, KUT_Connector:DF3A-3P-2DSA, symbol KRC_Conn3_SIG
- added P3: PORT, KUT_Connector:DF3A-5P-2DSA, symbol KRC_Conn5_SIG
- R11: footprint (none) -> Resistors_SMD:R_0603
- U6: symbol TWE-Lite -> TWE-Lite-RESCUE-RaSK_Generic-Rocket-Logger
Connections:
- net +3V3: now also P3.2 (VCC)
- net GND: now also P3.1 (GND)
- net LPS22HB_DRDY: now reaches U3.6 (INT_DRDY)
- net LPS22HB_DRDY: now also U1.59 (PB7)
- net BUZZ: now reaches U1.38 (PC7)
- net BUZZ: now also P3.5 (SIG3)
- net FPIN: now reaches U1.39 (PC8)
- net FPIN: now also P3.4 (SIG2)
- net TRIGSIG renamed TRIG
- net TRIG: now also P3.3 (SIG1)
- no-connect marks 89 -> 85
Other:
- moved on the sheet: R8, R9
Changed lines of the file:
@@
 EESchema Schematic File Version 2
+LIBS:RaSK_Generic-Rocket-Logger-rescue
 LIBS:power
 LIBS:device
@@
 	1    0    0    -1
 $EndComp
-NoConn ~ 2950 10000
 Text Label 3350 8550 0    60   ~ 0
 I2C2_SCL
@@
 STM_RESET
 $Comp
-L TWE-Lite U6
+L TWE-Lite-RESCUE-RaSK_Generic-Rocket-Logger U6
 U 1 1 596A8C77
 P 14350 8350
@@
 Text Label 6700 2650 2    60   ~ 0
 I2C1_SCL
-Text Label 6700 4250 2    60   ~ 0
+Text Label 6400 4250 2    60   ~ 0
 I2C2_SCL
-Text Label 6700 4350 2    60   ~ 0
+Text Label 6400 4350 2    60   ~ 0
 I2C2_SDA
 NoConn ~ 7600 3250
@@
 NoConn ~ 7600 3950
 NoConn ~ 7600 4050
-NoConn ~ 7600 4150
 NoConn ~ 7600 4450
 NoConn ~ 7600 4550
@@
 NoConn ~ 9700 2050
 NoConn ~ 9700 2350
-NoConn ~ 9700 2450
-NoConn ~ 9700 2550
 NoConn ~ 9700 2750
 NoConn ~ 9700 2850
@@
 L R_Small R8
 U 1 1 596DC09E
-P 6850 4050
-F 0 "R8" H 6880 4070 50  0000 L CNN
-F 1 "10k" H 6880 4010 50  0000 L CNN
-F 2 "Resistors_SMD:R_0603" H 6850 4050 50  0001 C CNN
-F 3 "" H 6850 4050 50  0001 C CNN
-	1    6850 4050
+P 6550 4050
+F 0 "R8" H 6580 4070 50  0000 L CNN
+F 1 "10k" H 6580 4010 50  0000 L CNN
+F 2 "Resistors_SMD:R_0603" H 6550 4050 50  0001 C CNN
+F 3 "" H 6550 4050 50  0001 C CNN
+	1    6550 4050
 	1    0    0    -1
 $EndComp
@@
 L R_Small R9
 U 1 1 596DC196
-P 7050 4050
-F 0 "R9" H 7080 4070 50  0000 L CNN
-F 1 "10k" H 7080 4010 50  0000 L CNN
-F 2 "Resistors_SMD:R_0603" H 7050 4050 50  0001 C CNN
-F 3 "" H 7050 4050 50  0001 C CNN
-	1    7050 4050
+P 6750 4050
+F 0 "R9" H 6780 4070 50  0000 L CNN
+F 1 "10k" H 6780 4010 50  0000 L CNN
+F 2 "Resistors_SMD:R_0603" H 6750 4050 50  0001 C CNN
+F 3 "" H 6750 4050 50  0001 C CNN
+	1    6750 4050
 	1    0    0    -1
 $EndComp
@@
 L +3.3V #PWR035
 U 1 1 596DC262
-P 6950 3850
-F 0 "#PWR035" H 6950 3700 50  0001 C CNN
-F 1 "+3.3V" H 6950 3990 50  0000 C CNN
-F 2 "" H 6950 3850 50  0001 C CNN
-F 3 "" H 6950 3850 50  0001 C CNN
-	1    6950 3850
+P 6650 3850
+F 0 "#PWR035" H 6650 3700 50  0001 C CNN
+F 1 "+3.3V" H 6650 3990 50  0000 C CNN
+F 2 "" H 6650 3850 50  0001 C CNN
+F 3 "" H 6650 3850 50  0001 C CNN
+	1    6650 3850
 	1    0    0    -1
 $EndComp
@@
 $EndComp
 $Comp
-L KRC_Conn3_SIG P3
-U 1 1 596EFFFB
-P 14850 2900
-F 0 "P3" H 14700 3150 60  0000 C CNN
-F 1 "TRIGOUT" H 14850 2630 60  0000 C CNN
-F 2 "KUT_Connector:DF3A-3P-2DSA" H 15050 2900 60  0001 C CNN
-F 3 "" H 15050 2900 60  0000 C CNN
-	1    14850 2900
-	1    0    0    -1
-$EndComp
-$Comp
 L +3.3V #PWR039
 U 1 1 596F132B
@@
 L GND #PWR040
 U 1 1 596F1522
-P 14450 3100
-F 0 "#PWR040" H 14450 2850 50  0001 C CNN
-F 1 "GND" H 14450 2950 50  0000 C CNN
-F 2 "" H 14450 3100 50  0001 C CNN
-F 3 "" H 14450 3100 50  0001 C CNN
-	1    14450 3100
+P 14450 3300
+F 0 "#PWR040" H 14450 3050 50  0001 C CNN
+F 1 "GND" H 14450 3150 50  0000 C CNN
+F 2 "" H 14450 3300 50  0001 C CNN
+F 3 "" H 14450 3300 50  0001 C CNN
+	1    14450 3300
 	1    0    0    -1
 $EndComp
 Text Label 14350 3000 2    60   ~ 0
-TRIGSIG
+TRIG
 Text Label 9700 2650 0    60   ~ 0
-TRIGSIG
+TRIG
 $Comp
 L GND #PWR041
@@
 F 0 "R11" H 3730 7070 50  0000 L CNN
 F 1 "1k" H 3730 7010 50  0000 L CNN
-F 2 "" H 3700 7050 50  0001 C CNN
+F 2 "Resistors_SMD:R_0603" H 3700 7050 50  0001 C CNN
 F 3 "" H 3700 7050 50  0001 C CNN
 	1    3700 7050
@@
 Connection ~ 6350 5250
 Wire Wire Line
-	6950 3850 6950 3900
-Wire Wire Line
-	6850 3900 7050 3900
-Wire Wire Line
-	6850 3900 6850 3950
-Wire Wire Line
-	7050 3900 7050 3950
-Connection ~ 6950 3900
-Wire Wire Line
-	7050 4150 7050 4350
-Wire Wire Line
-	6700 4350 7600 4350
-Wire Wire Line
-	6700 4250 7600 4250
-Wire Wire Line
-	6850 4250 6850 4150
-Connection ~ 6850 4250
-Connection ~ 7050 4350
+	6650 3850 6650 3900
+Wire Wire Line
+	6550 3900 6750 3900
+Wire Wire Line
+	6550 3900 6550 3950
+Wire Wire Line
+	6750 3900 6750 3950
+Connection ~ 6650 3900
+Wire Wire Line
+	6750 4150 6750 4350
+Wire Wire Line
+	6400 4350 7600 4350
+Wire Wire Line
+	6400 4250 7600 4250
+Wire Wire Line
+	6550 4250 6550 4150
+Connection ~ 6550 4250
+Connection ~ 6750 4350
 Wire Wire Line
 	6950 2250 6950 2300
@@
 	14550 2900 14650 2900
 Wire Wire Line
-	14450 3100 14450 2800
+	14450 2800 14450 3300
 Wire Wire Line
 	14450 2800 14650 2800
@@
 NoConn ~ 11500 10500
 NoConn ~ 11250 10500
+$Comp
+L KRC_Conn5_SIG P3
+U 1 1 599008CD
+P 14850 3000
+F 0 "P3" H 14725 3350 60  0000 C CNN
+F 1 "PORT" H 14850 2650 60  0000 C CNN
+F 2 "KUT_Connector:DF3A-5P-2DSA" H 15075 3000 60  0001 C CNN
+F 3 "" H 15075 3000 60  0000 C CNN
+	1    14850 3000
+	1    0    0    -1
+$EndComp
+Text Label 9700 2550 0    60   ~ 0
+FPIN
+Text Label 9700 2450 0    60   ~ 0
+BUZZ
+Text Label 14350 3100 2    60   ~ 0
+FPIN
+Text Label 14350 3200 2    60   ~ 0
+BUZZ
+Wire Wire Line
+	14350 3200 14650 3200
+Wire Wire Line
+	14650 3100 14350 3100
+Text Label 2950 10000 0    60   ~ 0
+LPS22HB_DRDY
+Text Label 7600 4150 2    60   ~ 0
+LPS22HB_DRDY
 $EndSCHEMATC

Commit message: board released
とりあえず完成品
Parts:
- added P4: UARTDebug, Pin_Headers:Pin_Header_Straight_1x04_Pitch2.54mm, symbol KRC_UARTModule
Connections:
- net BUZZ: now also P3.4 (SIG2), U1.39 (PC8); no longer P3.5 (SIG3), U1.38 (PC7)
- net FPIN: now also P3.5 (SIG3), U1.38 (PC7); no longer P3.4 (SIG2), U1.39 (PC8)
- net GND: now also P4.2 (GND)
- net SD_MISO: now also U1.22 (PA6); no longer U1.23 (PA7)
- net SD_MOSI: now also U1.23 (PA7); no longer U1.22 (PA6)
- net TWE_MIN: now also U1.56 (PB4), U6.8 (UART_Tx); no longer U1.55 (PB3), U6.9 (UART_Rx)
- net TWE_MOUT: now also U1.55 (PB3), U6.9 (UART_Rx); no longer U1.56 (PB4), U6.8 (UART_Tx)
- net Debug_MOUT: now reaches U1.51 (PC10)
- net Debug_MOUT: now also P4.4 (RXD)
- net Debug_MIN: now reaches U1.52 (PC11)
- net Debug_MIN: now also P4.3 (TXD)
- no-connect marks 85 -> 84
Changed lines of the file:
@@
 NoConn ~ 15200 8900
 NoConn ~ 15200 9000
+Text Label 15200 7750 0    60   ~ 0
+TWE_MOUT
 Text Label 15200 7650 0    60   ~ 0
-TWE_MOUT
-Text Label 15200 7750 0    60   ~ 0
 TWE_MIN
 NoConn ~ 13500 7650
@@
 	1    0    0    -1
 $EndComp
+Text Label 7600 2350 2    60   ~ 0
+SD_MISO
 Text Label 7600 2450 2    60   ~ 0
-SD_MISO
-Text Label 7600 2350 2    60   ~ 0
 SD_MOSI
 Text Label 7600 2250 2    60   ~ 0
@@
 	1    0    0    -1
 $EndComp
+Text Label 7600 3750 2    60   ~ 0
+TWE_MOUT
 Text Label 7600 3850 2    60   ~ 0
-TWE_MOUT
-Text Label 7600 3750 2    60   ~ 0
 TWE_MIN
 NoConn ~ 7600 3450
@@
 NoConn ~ 9700 2050
 NoConn ~ 9700 2350
-NoConn ~ 9700 2750
-NoConn ~ 9700 2850
 NoConn ~ 9700 2950
 NoConn ~ 9700 3050
@@
 	1    0    0    -1
 $EndComp
+Text Label 9700 2450 0    60   ~ 0
+FPIN
 Text Label 9700 2550 0    60   ~ 0
+BUZZ
+Text Label 14350 3200 2    60   ~ 0
 FPIN
-Text Label 9700 2450 0    60   ~ 0
-BUZZ
 Text Label 14350 3100 2    60   ~ 0
-FPIN
-Text Label 14350 3200 2    60   ~ 0
 BUZZ
 Wire Wire Line
@@
 Text Label 7600 4150 2    60   ~ 0
 LPS22HB_DRDY
+NoConn ~ 11650 3100
+$Comp
+L GND #PWR048
+U 1 1 5992172F
+P 11550 3500
+F 0 "#PWR048" H 11550 3250 50  0001 C CNN
+F 1 "GND" H 11550 3350 50  0000 C CNN
+F 2 "" H 11550 3500 50  0001 C CNN
+F 3 "" H 11550 3500 50  0001 C CNN
+	1    11550 3500
+	1    0    0    -1
+$EndComp
+Wire Wire Line
+	11550 3500 11550 3200
+Wire Wire Line
+	11550 3200 11650 3200
+Text Label 11450 3400 2    60   ~ 0
+Debug_MOUT
+Wire Wire Line
+	11450 3400 11650 3400
+Text Label 11450 3300 2    60   ~ 0
+Debug_MIN
+Wire Wire Line
+	11450 3300 11650 3300
+Text Label 9700 2850 0    60   ~ 0
+Debug_MIN
+Text Label 9700 2750 0    60   ~ 0
+Debug_MOUT
+$Comp
+L KRC_UARTModule P4
+U 1 1 599227DA
+P 11850 3250
+F 0 "P4" H 11800 3500 60  0000 C CNN
+F 1 "UARTDebug" H 11850 3000 60  0000 C CNN
+F 2 "Pin_Headers:Pin_Header_Straight_1x04_Pitch2.54mm" H 12075 3200 60  0001 C CNN
+F 3 "" H 12075 3200 60  0000 C CNN
+	1    11850 3250
+	1    0    0    -1
+$EndComp
 $EndSCHEMATC
